File: backplane.kicad_sch (KiCad schematic)
At the start: 85 parts, among them J3 CONN_2, P1 S100_FEMALE, P10 S100_FEMALE, P2 S100_FEMALE, P3 S100_FEMALE, P4 S100_FEMALE, P5 S100_FEMALE, P6 S100_FEMALE, P7 S100_FEMALE, P8 S100_FEMALE, P9 S100_FEMALE, Q1 TIP29, Q2 BC858, Q3 TIP30, Q4 BC848, U1 LM7301

Commit message: Update to rev A to provide active termination on all non-power lines.
Parts:
- removed C3, C5, C7: 0.01uF, backplane:C_0805, symbol backplane:C
- removed C4, C6, C8: 1uF, backplane:CP_0805, symbol backplane:C_Polarized
- removed R4, R5, R6, R7: 560, backplane:R_0805, symbol backplane:R
- removed RN21, RN22, RN23: 560, backplane:R_Array_Convex_4x1206, symbol backplane:R_Pack04
- added C10, C6, C8: 10nF, backplane:C_0805, symbol backplane:C
- added C5, C7, C9: 1uF, backplane:CP_0805, symbol backplane:C_Polarized
- added RN25, RN26, RN27, RN33, RN34, RN35, RN36, RN37, RN38, RN39, RN40, RN41, RN42, RN43, RN44, RN45, RN46: 560, backplane:R_Array_Convex_4x1206, symbol backplane:R_Pack04
- C4: renamed from C2; value 0.01uF -> 10nF
- renumbered C9 to C1, C10 to C2, C1 to C3, Q2 to Q1, Q1 to Q2, R12 to R10, R14 to R11, R15 to R12, R8 to R4, R10 to R5, R9 to R6, R11 to R7, R13 to R8, R16 to R9, RN25 to RN18, RN18 to RN19, RN26 to RN20, RN19 to RN21, RN27 to RN22, RN20 to RN23
Connections:
- net GND: now also C10.2, C5.2, C6.2, C7.2, C8.2, C9.2
- net VACT: now also RN24.1 (R1.1), RN24.2 (R2.1), RN24.3 (R3.1), RN24.4 (R4.1), RN28.1 (R1.1), RN28.2 (R2.1), RN28.3 (R3.1), RN28.4 (R4.1), RN29.1 (R1.1), RN29.2 (R2.1), RN29.3 (R3.1), RN29.4 (R4.1), RN30.1 (R1.1), RN30.2 (R2.1), RN30.3 (R3.1), RN30.4 (R4.1), RN31.1 (R1.1), RN31.2 (R2.1), RN31.3 (R3.1), RN31.4 (R4.1), RN32.1 (R1.1), RN32.2 (R2.1), RN32.3 (R3.1), RN32.4 (R4.1), C10.1, C5.1, C6.1, C7.1, C8.1, C9.1, RN25.1 (R1.1), RN25.2 (R2.1), RN25.3 (R3.1), RN25.4 (R4.1), RN26.1 (R1.1), RN26.2 (R2.1), RN26.3 (R3.1), RN26.4 (R4.1), RN27.1 (R1.1), RN27.2 (R2.1), RN27.3 (R3.1), RN27.4 (R4.1), RN33.1 (R1.1), RN33.2 (R2.1), RN33.3 (R3.1), RN33.4 (R4.1), RN34.1 (R1.1), RN34.2 (R2.1), RN34.3 (R3.1), RN34.4 (R4.1), RN35.1 (R1.1), RN35.2 (R2.1), RN35.3 (R3.1), RN35.4 (R4.1), RN36.1 (R1.1), RN36.2 (R2.1), RN36.3 (R3.1), RN36.4 (R4.1), RN37.1 (R1.1), RN37.2 (R2.1), RN37.3 (R3.1), RN37.4 (R4.1), RN38.1 (R1.1), RN38.2 (R2.1), RN38.3 (R3.1), RN38.4 (R4.1), RN39.1 (R1.1), RN39.2 (R2.1), RN39.3 (R3.1), RN39.4 (R4.1), RN40.1 (R1.1), RN40.2 (R2.1), RN40.3 (R3.1), RN40.4 (R4.1), RN41.1 (R1.1), RN41.2 (R2.1), RN41.3 (R3.1), RN41.4 (R4.1), RN42.1 (R1.1), RN42.2 (R2.1), RN42.3 (R3.1), RN42.4 (R4.1), RN43.1 (R1.1), RN43.2 (R2.1), RN43.3 (R3.1), RN43.4 (R4.1), RN44.1 (R1.1), RN44.2 (R2.1), RN44.3 (R3.1), RN44.4 (R4.1), RN45.1 (R1.1), RN45.2 (R2.1), RN45.3 (R3.1), RN45.4 (R4.1), RN46.1 (R1.1), RN46.2 (R2.1), RN46.3 (R3.1), RN46.4 (R4.1); no longer RN24.5 (R4.2), RN24.6 (R3.2), RN24.7 (R2.2), RN24.8 (R1.2), RN28.5 (R4.2), RN28.6 (R3.2), RN28.7 (R2.2), RN28.8 (R1.2), RN29.5 (R4.2), RN29.6 (R3.2), RN29.7 (R2.2), RN29.8 (R1.2), RN30.5 (R4.2), RN30.6 (R3.2), RN30.7 (R2.2), RN30.8 (R1.2), RN31.5 (R4.2), RN31.6 (R3.2), RN31.7 (R2.2), RN31.8 (R1.2), RN32.5 (R4.2), RN32.6 (R3.2), RN32.7 (R2.2), RN32.8 (R1.2)
- net bus_003: now also RN1.1 (R1.1), RN24.8 (R1.2)
- net bus_004: now also RN1.3 (R3.1), RN24.6 (R3.2)
- net bus_005: now also RN2.1 (R1.1), RN25.8 (R1.2)
- net bus_006: now also RN2.3 (R3.1), RN25.6 (R3.2)
- net bus_007: now also RN3.1 (R1.1), RN26.8 (R1.2)
- net bus_008: now also RN3.3 (R3.1), RN26.6 (R3.2)
- net bus_009: now also RN4.1 (R1.1), RN27.8 (R1.2)
- net bus_010: now also RN4.3 (R3.1), RN27.6 (R3.2)
- net bus_011: now also RN28.8 (R1.2), RN5.1 (R1.1)
- net bus_012: now also RN28.6 (R3.2), RN5.3 (R3.1)
- net bus_013: now also RN29.8 (R1.2), RN6.1 (R1.1); no longer RN18.3 (R3.1), RN2.2 (R2.1)
- net bus_014: now also RN29.6 (R3.2), RN6.3 (R3.1)
- net bus_015: now also RN30.8 (R1.2), RN7.1 (R1.1); no longer RN19.4 (R4.1), RN3.1 (R1.1)
- net bus_016: now also RN30.6 (R3.2), RN7.3 (R3.1); no longer RN19.2 (R2.1), RN3.3 (R3.1)
- net bus_017: now also RN31.8 (R1.2), RN8.1 (R1.1); no longer RN19.1 (R1.1), RN3.4 (R4.1)
- net bus_018: now also RN31.6 (R3.2), RN8.3 (R3.1)
- net bus_019: now also RN32.8 (R1.2), RN9.1 (R1.1)
- net bus_021: now also RN32.5 (R4.2), RN9.3 (R3.1); no longer RN20.1 (R1.1), RN4.3 (R3.1)
- net bus_022: now also RN10.1 (R1.1), RN33.7 (R2.2)
- net bus_023: now also RN10.3 (R3.1), RN33.5 (R4.2)
- net bus_024: now also RN11.1 (R1.1), RN34.7 (R2.2); no longer RN21.4 (R4.1), RN5.1 (R1.1)
- net bus_025: now also RN11.3 (R3.1), RN34.5 (R4.2); no longer RN21.2 (R2.1), RN5.2 (R2.1)
- net bus_026: now also RN12.1 (R1.1), RN35.8 (R1.2); no longer RN21.1 (R1.1), RN5.3 (R3.1)
- net bus_027: now also RN12.3 (R3.1), RN35.6 (R3.2); no longer RN22.3 (R3.1), RN6.1 (R1.1)
- net bus_028: now also RN13.1 (R1.1), RN36.8 (R1.2); no longer RN22.1 (R1.1), RN6.3 (R3.1)
- net bus_029: now also RN13.3 (R3.1), RN36.6 (R3.2); no longer RN23.3 (R3.1), RN7.1 (R1.1)
- net bus_030: now also RN14.1 (R1.1), RN37.8 (R1.2); no longer RN23.1 (R1.1), RN7.3 (R3.1)
- net bus_031: now also RN14.3 (R3.1), RN37.6 (R3.2); no longer RN28.3 (R3.1), RN8.1 (R1.1)
- net bus_032: now also RN15.1 (R1.1), RN38.8 (R1.2); no longer RN28.1 (R1.1), RN8.3 (R3.1)
- net bus_033: now also RN15.3 (R3.1), RN38.6 (R3.2); no longer RN9.2 (R2.1)
- net bus_034: now also RN16.1 (R1.1), RN39.8 (R1.2); no longer RN9.4 (R4.1)
- net bus_035: now also RN16.3 (R3.1), RN39.6 (R3.2); no longer RN10.2 (R2.1), RN29.4 (R4.1)
- net bus_036: now also RN17.1 (R1.1), RN40.8 (R1.2); no longer RN10.4 (R4.1), RN29.2 (R2.1)
- net bus_037: now also RN17.3 (R3.1), RN40.6 (R3.2); no longer RN11.2 (R2.1)
- net bus_038: now also RN18.1 (R1.1), RN41.8 (R1.2); no longer RN11.4 (R4.1)
- net bus_039: now also RN18.3 (R3.1), RN41.6 (R3.2); no longer RN12.2 (R2.1), RN30.4 (R4.1)
- net bus_040: now also RN19.1 (R1.1), RN42.8 (R1.2); no longer RN12.4 (R4.1), RN30.2 (R2.1)
- net bus_041: now also RN19.3 (R3.1), RN42.6 (R3.2); no longer RN13.2 (R2.1)
- net bus_042: now also RN20.1 (R1.1), RN43.8 (R1.2); no longer RN13.4 (R4.1)
- net bus_043: now also RN20.3 (R3.1), RN43.6 (R3.2); no longer RN14.2 (R2.1), RN31.4 (R4.1)
- net bus_044: now also RN21.1 (R1.1), RN44.8 (R1.2); no longer RN14.4 (R4.1), RN31.2 (R2.1)
- net bus_045: now also RN21.3 (R3.1), RN44.6 (R3.2); no longer RN15.2 (R2.1), RN24.4 (R4.1)
- net bus_046: now also RN22.1 (R1.1), RN45.8 (R1.2); no longer RN15.4 (R4.1), RN24.2 (R2.1)
- net bus_047: now also RN22.3 (R3.1), RN45.6 (R3.2); no longer RN16.2 (R2.1), RN32.4 (R4.1)
- net bus_048: now also RN23.1 (R1.1), RN46.8 (R1.2); no longer RN16.3 (R3.1), RN32.2 (R2.1)
- net bus_049: now also RN23.3 (R3.1), RN46.6 (R3.2)
- net bus_054: now also RN1.2 (R2.1), RN24.7 (R2.2)
- net bus_055: now also RN1.4 (R4.1), RN24.5 (R4.2)
- net bus_056: now also RN2.2 (R2.1), RN25.7 (R2.2)
- net bus_057: now also RN2.4 (R4.1), RN25.5 (R4.2)
- net bus_058: now also RN3.2 (R2.1), RN26.7 (R2.2); no longer RN1.1 (R1.1), RN17.4 (R4.1)
- net bus_059: now also RN3.4 (R4.1), RN26.5 (R4.2); no longer RN1.2 (R2.1), RN17.3 (R3.1)
- net bus_060: now also RN4.2 (R2.1), RN27.7 (R2.2)
- net bus_061: now also RN4.4 (R4.1), RN27.5 (R4.2); no longer RN1.3 (R3.1), RN17.2 (R2.1)
- net bus_062: now also RN28.7 (R2.2), RN5.2 (R2.1); no longer RN1.4 (R4.1), RN17.1 (R1.1)
- net bus_063: now also RN28.5 (R4.2), RN5.4 (R4.1); no longer RN18.4 (R4.1), RN2.1 (R1.1)
- net bus_064: now also RN29.7 (R2.2), RN6.2 (R2.1); no longer RN18.2 (R2.1), RN2.3 (R3.1)
- net bus_065: now also RN29.5 (R4.2), RN6.4 (R4.1); no longer RN18.1 (R1.1), RN2.4 (R4.1)
- net bus_066: now also RN30.7 (R2.2), RN7.2 (R2.1); no longer RN19.3 (R3.1), RN3.2 (R2.1)
- net bus_067: now also RN30.5 (R4.2), RN7.4 (R4.1)
- net bus_068: now also RN31.7 (R2.2), RN8.2 (R2.1); no longer RN20.4 (R4.1), RN4.1 (R1.1)
- net bus_069: now also RN31.5 (R4.2), RN8.4 (R4.1); no longer RN20.3 (R3.1), RN4.2 (R2.1)
- net bus_071: now also RN32.6 (R3.2), RN9.4 (R4.1); no longer RN20.2 (R2.1), RN4.4 (R4.1)
- net bus_072: now also RN10.2 (R2.1), RN33.8 (R1.2)
- net bus_073: now also RN10.4 (R4.1), RN33.6 (R3.2)
- net bus_074: now also RN11.2 (R2.1), RN34.8 (R1.2)
- net bus_075: now also RN11.4 (R4.1), RN34.6 (R3.2)
- net bus_076: now also RN12.2 (R2.1), RN35.7 (R2.2); no longer RN21.3 (R3.1), RN5.4 (R4.1)
- net bus_077: now also RN12.4 (R4.1), RN35.5 (R4.2); no longer RN22.4 (R4.1), RN6.2 (R2.1)
- net bus_078: now also RN13.2 (R2.1), RN36.7 (R2.2); no longer RN22.2 (R2.1), RN6.4 (R4.1)
- net bus_079: now also RN13.4 (R4.1), RN36.5 (R4.2); no longer RN23.4 (R4.1), RN7.2 (R2.1)
- net bus_080: now also RN14.2 (R2.1), RN37.7 (R2.2); no longer RN23.2 (R2.1), RN7.4 (R4.1)
- net bus_081: now also RN14.4 (R4.1), RN37.5 (R4.2); no longer RN28.4 (R4.1), RN8.2 (R2.1)
- net bus_082: now also RN15.2 (R2.1), RN38.7 (R2.2); no longer RN28.2 (R2.1), RN8.4 (R4.1)
- net bus_083: now also RN15.4 (R4.1), RN38.5 (R4.2); no longer RN9.1 (R1.1)
- net bus_084: now also RN16.2 (R2.1), RN39.7 (R2.2); no longer RN9.3 (R3.1)
- net bus_085: now also RN16.4 (R4.1), RN39.5 (R4.2); no longer RN10.1 (R1.1), RN29.3 (R3.1)
- net bus_086: now also RN17.2 (R2.1), RN40.7 (R2.2); no longer RN10.3 (R3.1), RN29.1 (R1.1)
- net bus_087: now also RN17.4 (R4.1), RN40.5 (R4.2); no longer RN11.1 (R1.1)
- net bus_088: now also RN18.2 (R2.1), RN41.7 (R2.2); no longer RN11.3 (R3.1)
- net bus_089: now also RN18.4 (R4.1), RN41.5 (R4.2); no longer RN12.1 (R1.1), RN30.3 (R3.1)
- net bus_090: now also RN19.2 (R2.1), RN42.7 (R2.2); no longer RN12.3 (R3.1), RN30.1 (R1.1)
- net bus_091: now also RN19.4 (R4.1), RN42.5 (R4.2); no longer RN13.1 (R1.1)
- net bus_092: now also RN20.2 (R2.1), RN43.7 (R2.2); no longer RN13.3 (R3.1)
- net bus_093: now also RN20.4 (R4.1), RN43.5 (R4.2); no longer RN14.1 (R1.1), RN31.3 (R3.1)
- net bus_094: now also RN21.2 (R2.1), RN44.7 (R2.2); no longer RN14.3 (R3.1), RN31.1 (R1.1)
- net bus_095: now also RN21.4 (R4.1), RN44.5 (R4.2); no longer RN15.1 (R1.1), RN24.3 (R3.1)
- net bus_096: now also RN22.2 (R2.1), RN45.7 (R2.2); no longer RN15.3 (R3.1), RN24.1 (R1.1)
- net bus_097: now also RN22.4 (R4.1), RN45.5 (R4.2); no longer RN16.1 (R1.1), RN32.3 (R3.1)
- net bus_098: now also RN23.2 (R2.1), RN46.7 (R2.2)
- net bus_099: now also RN23.4 (R4.1), RN46.5 (R4.2); no longer RN16.4 (R4.1), RN32.1 (R1.1)
- no-connect marks 0 -> 2
Other:
- title: Active Backplane -> 10-slot S-100 Bus Active Backplane
- moved on the sheet: C1, C2, C3, C4, D1, D2, D3, D4, Q1, Q2, Q3, Q4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
